File: MainBoard/followLineMain.brd (EAGLE design)
At the start: 94.9 x 53.1 mm, 32 parts, among them IC1 L298, J1 DCJ0202, X1 332-02, X2 332-02

Commit message: Corrected some aspects of the boards and another version of the SensorBoard
Routing:
- net GND: track 268.7 -> 281.1 mm
- net PWM4: track 54.3 -> 61.9 mm
- net VIN: track 67.3 -> 72.1 mm
- net PWM3: track 30.1 -> 33.1 mm
- net PWM2: track 30.1 -> 32.2 mm
- net VBAT: track 117.0 -> 116.4 mm
