File: MainBoard/v2/followLineMain.brd (EAGLE design)
At the start: 94.9 x 53.1 mm, 32 parts, among them IC1 L298, J1 DCJ0202, X1 332-02, X2 332-02

Commit message: Corrected some aspects of the boards and another version of the SensorBoard
Routing:
- net GND: track 260.7 -> 285.5 mm
- net VIN: track 67.3 -> 70.9 mm
- net OUT3: track 25.2 -> 26.9 mm
- net VBAT: track 116.5 -> 117.9 mm
- net OUT2: track 30.5 -> 29.9 mm
