File: SensorBoard/v2/followLineSensor.brd (EAGLE design)
At the start: 102.5 x 31.7 mm, 29 parts

Commit message: Corrected some aspects of the boards and another version of the SensorBoard
Parts:
- removed JP1, JP2, JP3, JP4, JP5: (no value), pinhead:1X01
- removed JP6: (no value), pinhead:1X02
- added SV1: (no value), con-lstb:MA07-1
- moved R1 17.8 mm to (45.7, 63.4), turned to 0 degrees
- moved LED1 14.8 mm to (47.7, 67.6)
- moved C1 8.37 mm to (40.0, 56.6)
- moved IR0 5.68 mm to (14.0, 44.5)
- moved L0 5.68 mm to (6.35, 44.5)
- moved IR4 5.68 mm to (88.9, 44.5)
- moved L4 5.68 mm to (81.3, 44.5)
- moved RIR0 5.08 mm to (14.0, 53.3)
- moved RL0 5.08 mm to (6.35, 53.3)
- moved RIR4 5.08 mm to (88.9, 53.3)
- moved RL4 5.08 mm to (81.3, 53.3)
- moved IR1 2.84 mm to (35.6, 44.5)
- moved L1 2.84 mm to (27.9, 44.5)
- moved IR3 2.84 mm to (68.6, 44.5)
- moved L3 2.84 mm to (61.0, 44.5)
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Connections:
- net A0: now also SV1.5; no longer JP5.1
- net A1: now also SV1.4; no longer JP4.1
- net A2: now also SV1.3; no longer JP3.1
- net A3: now also SV1.2; no longer JP2.1
- net A4: now also SV1.1; no longer JP1.1
- net GND: now also SV1.6; no longer JP6.1
- net VBAT: now also SV1.7; no longer JP6.2
Routing:
- net A0: track 14.1 -> 98.5 mm, vias 0 -> 1
- net A1: track 16.1 -> 81.2 mm, vias 0 -> 1
- net A2: track 14.1 -> 49.2 mm, vias 0 -> 1
- net A3: track 15.9 -> 43.1 mm, vias 0 -> 1
- net GND: track 187.7 -> 213.6 mm, vias 0 -> 1
- net A4: track 16.6 -> 29.4 mm, vias 0 -> 1
- net VBAT: track 115.9 -> 125.4 mm, vias 0 -> 1
- net N$21: track 8.76 -> 6.22 mm
- net N$20: track 8.76 -> 6.22 mm
- net N$19: track 8.76 -> 6.22 mm
- net N$18: track 8.76 -> 6.22 mm
- net N$17: track 8.76 -> 6.22 mm
- net N$2: track 4.88 -> 5.51 mm
Other:
- board size 102.5 x 31.7 mm -> 102.5 x 34.3 mm

Commit message: Another better versions of the boards done
Parts:
- removed C1: 100nF, rcl:C0805
- added C2: 1uF, rcl:C1206
- moved L4 13.5 mm to (94.8, 44.4)
- moved RL4 13.5 mm to (94.8, 53.2)
- moved IR4 12.7 mm to (101.6, 44.4)
- moved RIR4 12.7 mm to (101.6, 53.2)
- moved R1 7.61 mm to (53.3, 63.0)
- moved IR0 6.60 mm to (7.37, 44.4)
- moved RIR0 6.60 mm to (7.37, 53.2)
- moved RL0 6.30 mm to (0.05, 53.2)
- moved L0 6.30 mm to (0.05, 44.5)
- moved SV1 2.95 mm to (85.2, 64.6)
- moved IR3 2.70 mm to (71.3, 44.4)
- moved L2 2.70 mm to (54.8, 44.4)
- moved RIR3 2.70 mm to (71.3, 53.2)
- moved RL2 2.70 mm to (54.8, 53.2)
- moved L1 2.70 mm to (30.6, 44.4)
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Connections:
- net GND: now also C2.2; no longer C1.2
- net VBAT: now also C2.1; no longer C1.1
Routing:
- net GND: track 213.6 -> 312.8 mm
- net VBAT: track 125.4 -> 177.3 mm
- net N$2: track 5.51 -> 11.0 mm
- net A0: track 98.5 -> 104.0 mm
- net A2: track 49.2 -> 46.4 mm
- net A1: track 81.2 -> 80.5 mm
- net A4: track 29.4 -> 30.1 mm
Other:
- board size 102.5 x 34.3 mm -> 112.7 x 31.1 mm
