File: SensorBoard/v2/followLineSensor.sch (EAGLE design)
At the start: 24 parts

Commit message: Another better versions of the boards done
Parts:
- removed C1: 100nF, rcl:C-EUC0805
- added C2: 1uF, rcl:C-EUC1206
Connections:
- net GND: now also C2.2; no longer C1.2
- net VBAT: now also C2.1; no longer C1.1
Changed lines of the file:
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@@
 <part name="R1" library="rcl" deviceset="R-US_" device="R0805" value="820"/>
 <part name="LED1" library="led" deviceset="LED" device="SML0805" value="green"/>
-<part name="C1" library="rcl" deviceset="C-EU" device="C0805" value="100nF"/>
 <part name="SV1" library="con-lstb" deviceset="MA07-1" device=""/>
+<part name="C2" library="rcl" deviceset="C-EU" device="C1206" value="1uF"/>
 </parts>
 <sheets>
@@
 <instance part="R1" gate="G$1" x="132.08" y="96.52" rot="R90"/>
 <instance part="LED1" gate="G$1" x="132.08" y="83.82"/>
-<instance part="C1" gate="G$1" x="119.38" y="91.44"/>
 <instance part="SV1" gate="1" x="-63.5" y="86.36"/>
+<instance part="C2" gate="G$1" x="119.38" y="91.44"/>
 </instances>
 <busses>
@@
 </segment>
 <segment>
-<pinref part="C1" gate="G$1" pin="1"/>
 <wire x1="119.38" y1="93.98" x2="119.38" y2="99.06" width="0.1524" layer="91"/>
 <label x="119.38" y="99.06" size="1.778" layer="95" rot="R90" xref="yes"/>
+<pinref part="C2" gate="G$1" pin="1"/>
 </segment>
 <segment>
@@
 </segment>
 <segment>
-<pinref part="C1" gate="G$1" pin="2"/>
 <wire x1="119.38" y1="86.36" x2="119.38" y2="81.28" width="0.1524" layer="91"/>
 <label x="119.38" y="81.28" size="1.778" layer="95" rot="R270" xref="yes"/>
+<pinref part="C2" gate="G$1" pin="2"/>
 </segment>
 <segment>
